File: vm-digital/stack DIP/stack DIP.kicad_sch (KiCad schematic)
At the start: 7 parts, among them J1 Conn_01x11_Pin, J2 Conn_01x11_Pin, U1 74LS151, U2 74LS151, U3 74LS151, U4 74LS151, U5 74LS151

Commit message: stack-dip
Parts:
- removed U1, U3, U4, U5: 74LS151, Package_SO:TSSOP-16_4.4x5mm_P0.65mm, symbol 74xx:74LS151
- added C1, C10, C2, C3, C4, C5, C6, C7, C8, C9: C_Small, Capacitor_SMD:C_0402_1005Metric, symbol Device:C_Small
- added U1: 74LS157, Package_DFN_QFN:DHVQFN-16-1EP_2.5x3.5mm_P0.5mm_EP1x2mm, symbol 74xx:74LS157
- added U3, U4: 74HC74, Package_DFN_QFN:DHVQFN-14-1EP_2.5x3mm_P0.5mm_EP1x1.5mm, symbol 74xx:74HC74
- added U6: 7408, Package_DFN_QFN:DHVQFN-14-1EP_2.5x3mm_P0.5mm_EP1x1.5mm, symbol 74xx_IEEE:7408
- U2: footprint Package_SO:TSSOP-16_4.4x5mm_P0.65mm -> Package_DFN_QFN:DHVQFN-16-1EP_2.5x3.5mm_P0.5mm_EP1x2mm
Other:
- moved on the sheet: U2
